File: hardware/nes-dev-cart.kicad_pcb (KiCad board)
At the start: 4 copper layers, 100 x 110 mm, 39 parts, among them J1 NES_72Pin, J2 DF40C-60DS, J3 DF40C-60DS, J4 USB_C, J5 JTAG, J6 EXPANSION, SW1 RESET, U1 74ALVC164245, U2 74ALVC164245, U3 74ALVC164245, U4 74ALVC164245, U5 FT2232HL, Y1 12MHz

Commit message: NES-DEV-CART v4.1: 8MB PSRAM, updated production files, website
- Updated KiCad PCB/schematic with 8MB SPI PSRAM (APS6404L)
- Regenerated gerbers, BOM, and CPL for v4.1
- Added product website (nesos.dev)
- Updated README with v4.1 specs
- Added GitHub link to website footer

Co-Authored-By: Claude Opus 4.6 <noreply@anthropic.com>
Parts:
- added C19: 100nF, Capacitor_SMD:C_0805_2012Metric, F.Cu at (160.0, 108.0)
- added C20: 10uF, Capacitor_SMD:C_0805_2012Metric, F.Cu at (160.0, 122.0)
- added U6: APS6404L, Package_SO:SOIC-8_3.9x4.9mm_P1.27mm, F.Cu at (160.0, 115.0)
Connections:
- J1 pad 53: /EXP_7 -> EXP_7
- J1 pad 54: /EXP_6 -> EXP_6
- J2 pad 25: /FPGA_DONE -> /PSRAM_CLK
- J2 pad 30: /EXP_6_3V3 -> /PSRAM_~{CS}
- J2 pad 32: /EXP_7_3V3 -> /PSRAM_SIO2
- J3 pad 22: /EXP_GPIO0 -> /PSRAM_SIO0
- J3 pad 24: /EXP_GPIO1 -> /PSRAM_SIO1
- J3 pad 36: /EXP_GPIO2 -> /PSRAM_SIO3
- J6 pad 1: /EXP_GPIO0 -> GND
- J6 pad 2: /EXP_GPIO1 -> GND
- J6 pad 3: /EXP_GPIO2 -> GND
- R5 pad 1: /FPGA_DONE -> +3V3
- U4 pad 19: /EXP_6 -> (no net)
- U4 pad 22: /EXP_7 -> (no net)
- U4 pad 27: /EXP_7_3V3 -> (no net)
- U4 pad 30: /EXP_6_3V3 -> (no net)
Routing:
- net /PSRAM_SIO3: track 0.00 -> 63.5 mm, vias 0 -> 2
- net /PSRAM_SIO0: track 0.00 -> 62.0 mm, vias 0 -> 2
- net /PSRAM_SIO1: track 0.00 -> 57.5 mm, vias 0 -> 2
- net /PSRAM_SIO2: track 0.00 -> 51.6 mm, vias 0 -> 2
- net /EXP_7_3V3: track 51.5 -> 0.00 mm, vias 1 -> 0
- net /EXP_6_3V3: track 51.5 -> 0.00 mm, vias 1 -> 0
- net /FPGA_DONE: track 49.2 -> 0.00 mm, vias 2 -> 0
- net /EXP_GPIO0: track 49.1 -> 0.00 mm, vias 1 -> 0
- net /EXP_GPIO2: track 46.1 -> 0.00 mm, vias 1 -> 0
- net /PSRAM_CLK: track 0.00 -> 46.0 mm, vias 0 -> 2
- net /EXP_GPIO1: track 45.5 -> 0.00 mm, vias 1 -> 0
- net /PSRAM_~{CS}: track 0.00 -> 40.7 mm, vias 0 -> 2
- net +3V3: track 340.2 -> 367.2 mm, vias 5 -> 3
- net /CPU_A1: track 54.5 -> 30.1 mm, vias 2 -> 0
- net /CPU_A7: track 20.6 -> 44.9 mm
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