File: hardware/nes-dev-cart.kicad_sch (KiCad schematic)
At the start: 38 parts, among them J2 DF40C-60DS, J3 DF40C-60DS, J4 USB_C, J5 JTAG, J6 EXPANSION, SW1 RESET, U1 74ALVC164245, U2 74ALVC164245, U3 74ALVC164245, U4 74ALVC164245, U5 FT2232HL, Y1 12MHz

Commit message: NES-DEV-CART v4.1: 8MB PSRAM, updated production files, website
- Updated KiCad PCB/schematic with 8MB SPI PSRAM (APS6404L)
- Regenerated gerbers, BOM, and CPL for v4.1
- Added product website (nesos.dev)
- Updated README with v4.1 specs
- Added GitHub link to website footer

Co-Authored-By: Claude Opus 4.6 <noreply@anthropic.com>
Parts:
- added C19: 100nF, symbol Device:C
- added C20: 10uF, symbol Device:C
- added U6: APS6404L, symbol Memory_RAM:APS6404L-3SQRx-SN
Connections:
- net +3V3: now also R5.1, C19.1, C20.1, U6.8 (VDD)
- net GND: now also J6.1 (Pin_1), J6.2 (Pin_2), J6.3 (Pin_3), C19.2, C20.2, U6.4 (VSS)
- net EXP_6: no longer names the net of U4.19 (2B4)
- net EXP_6_3V3: no longer names the net of U4.30 (2A4)
- net EXP_6_3V3: no longer J2.30 (Pin_30)
- net EXP_7: no longer names the net of U4.22 (2B6)
- net EXP_7_3V3: no longer names the net of U4.27 (2A6)
- net EXP_7_3V3: no longer J2.32 (Pin_32)
- net EXP_GPIO0 renamed PSRAM_SIO0
- net PSRAM_SIO0: now also U6.5 (SI/SIO0); no longer J6.1 (Pin_1)
- net EXP_GPIO1 renamed PSRAM_SIO1
- net PSRAM_SIO1: now also U6.2 (SO/SIO1); no longer J6.2 (Pin_2)
- net EXP_GPIO2 renamed PSRAM_SIO3
- net PSRAM_SIO3: now also U6.7 (SIO3); no longer J6.3 (Pin_3)
- net FPGA_DONE renamed PSRAM_CLK
- net PSRAM_CLK: now also U6.6 (SCLK); no longer R5.1
- new net PSRAM_SIO2: J2.32 (Pin_32), U6.3 (SIO2)
- new net PSRAM_~{CS}: J2.30 (Pin_30), U6.1 (~{CE})
- no-connect marks 53 -> 57
